Commit message: Update frame configuration to match Gazebo simulation
- Updated robot.urdf.xacro with correct TF tree structure
- Added unilidar_link intermediate frame matching Gazebo model
- Set sensor frames /unilidar_lidar and /unilidar_imu as children of unilidar_link
- Updated params.yaml lidarFrame to /unilidar_lidar
- Frame hierarchy now matches: base_link -> unilidar_link -> sensor frames

File: config/robot.urdf.xacro (robot description, xacro)
@@ -2,33 +2,28 @@
 <robot name="lio" xmlns:xacro="http://tixiaoshan.github.io/">
   <xacro:property name="PI" value="3.1415926535897931" />
-  <link name="chassis_link"></link>
+  <!-- Base link - root of the robot -->
   <link name="base_link"></link>
-  <joint name="base_link_joint" type="fixed">
-    <parent link="base_link"/>
-    <child link="chassis_link" />
+  <!-- Unilidar sensor assembly link - matches Gazebo unilidar_link -->
+  <!-- This represents the physical sensor housing containing both LiDAR and IMU -->
+  <link name="unilidar_link"></link>
+  <joint name="unilidar_joint" type="fixed">
+    <parent link="base_link" />
+    <child link="unilidar_link" />
+    <origin xyz="0 0 0.065" rpy="0 0 0" />
+  </joint>
+  <!-- LiDAR sensor frame - matches Gazebo sensor frame_id -->
+  <!-- Co-located with unilidar_link (no offset) -->
+  <link name="/unilidar_lidar"></link>
+  <joint name="lidar_joint" type="fixed">
+    <parent link="unilidar_link" />
+    <child link="/unilidar_lidar" />
     <origin xyz="0 0 0" rpy="0 0 0" />
   </joint>
-  <link name="lidar_link"> </link>
-  <joint name="lidar_joint" type="fixed">
-    <parent link="base_link" />
-    <child link="lidar_link" />
-    <origin xyz="0 0 0" rpy="0 0 0" />
-  </joint>
-  <link name="imu_link"> </link>
+  <!-- IMU sensor frame - matches Gazebo sensor frame_id -->
+  <!-- Co-located with LiDAR in the same sensor housing -->
+  <link name="/unilidar_imu"></link>
   <joint name="imu_joint" type="fixed">
-    <parent link="chassis_link" />
-    <child link="imu_link" />
-    <origin xyz="0 0 0" rpy="0 0 0" />
-  </joint>
-  <link name="laser_sensor_frame"> </link>
-  <joint name="laser_joint" type="fixed">
-    <parent link="imu_link" />
-    <child link="laser_sensor_frame" />
-    <origin xyz="0 0 0" rpy="0 0 0" />
-  </joint>
-  <link name="navsat_link"> </link>
-  <joint name="navsat_joint" type="fixed">
-    <parent link="chassis_link" />
-    <child link="navsat_link" />
+    <parent link="unilidar_link" />
+    <child link="/unilidar_imu" />
     <origin xyz="0 0 0" rpy="0 0 0" />
   </joint>

Commit message: feat: Add `use_sim_time` launch argument to nodes, update `lidarFrame` parameter, and set `sensor` type to `velodyne`.

File: config/robot.urdf.xacro (robot description, xacro)
@@ -14,16 +14,16 @@
   <!-- LiDAR sensor frame - matches Gazebo sensor frame_id -->
   <!-- Co-located with unilidar_link (no offset) -->
-  <link name="/unilidar_lidar"></link>
+  <link name="unilidar_lidar"></link>
   <joint name="lidar_joint" type="fixed">
     <parent link="unilidar_link" />
-    <child link="/unilidar_lidar" />
+    <child link="unilidar_lidar" />
     <origin xyz="0 0 0" rpy="0 0 0" />
   </joint>
   <!-- IMU sensor frame - matches Gazebo sensor frame_id -->
   <!-- Co-located with LiDAR in the same sensor housing -->
-  <link name="/unilidar_imu"></link>
+  <link name="unilidar_imu"></link>
   <joint name="imu_joint" type="fixed">
     <parent link="unilidar_link" />
-    <child link="/unilidar_imu" />
+    <child link="unilidar_imu" />
     <origin xyz="0 0 0" rpy="0 0 0" />
   </joint>

Commit message: feat: Rename sensor topics and frames from unilidar to lidar, and remove static world-to-map transform.

File: config/robot.urdf.xacro (robot description, xacro)
@@ -4,26 +4,26 @@
   <!-- Base link - root of the robot -->
   <link name="base_link"></link>
-  <!-- Unilidar sensor assembly link - matches Gazebo unilidar_link -->
+  <!-- GzLidar sensor assembly link - matches Gazebo gzlidar_link -->
   <!-- This represents the physical sensor housing containing both LiDAR and IMU -->
-  <link name="unilidar_link"></link>
-  <joint name="unilidar_joint" type="fixed">
+  <link name="lidar_link"></link>
+  <joint name="lidar_joint" type="fixed">
     <parent link="base_link" />
-    <child link="unilidar_link" />
+    <child link="lidar_link" />
     <origin xyz="0 0 0.065" rpy="0 0 0" />
   </joint>
   <!-- LiDAR sensor frame - matches Gazebo sensor frame_id -->
-  <!-- Co-located with unilidar_link (no offset) -->
-  <link name="unilidar_lidar"></link>
-  <joint name="lidar_joint" type="fixed">
-    <parent link="unilidar_link" />
-    <child link="unilidar_lidar" />
+  <!-- Co-located with lidar_link (no offset) -->
+  <link name="lidar_cloud"></link>
+  <joint name="lidar_cloud_joint" type="fixed">
+    <parent link="lidar_link" />
+    <child link="lidar_cloud" />
     <origin xyz="0 0 0" rpy="0 0 0" />
   </joint>
   <!-- IMU sensor frame - matches Gazebo sensor frame_id -->
   <!-- Co-located with LiDAR in the same sensor housing -->
-  <link name="unilidar_imu"></link>
-  <joint name="imu_joint" type="fixed">
-    <parent link="unilidar_link" />
-    <child link="unilidar_imu" />
+  <link name="lidar_imu"></link>
+  <joint name="lidar_imu_joint" type="fixed">
+    <parent link="lidar_link" />
+    <child link="lidar_imu" />
     <origin xyz="0 0 0" rpy="0 0 0" />
   </joint>

Commit message: fix: Update extrinsic RPY values for improved sensor alignment in params.yaml and correct joint origin RPY in robot.urdf.xacro

File: config/robot.urdf.xacro (robot description, xacro)
@@ -10,5 +10,5 @@
     <parent link="base_link" />
     <child link="lidar_link" />
-    <origin xyz="0 0 0.065" rpy="0 0 0" />
+    <origin xyz="0 0 0.065" rpy="0 0.78539816339 0" />
   </joint>
   <!-- LiDAR sensor frame - matches Gazebo sensor frame_id -->
